Commit message: Updating to add collisions to gripper links

File: baxter_description/urdf/baxter.urdf (robot description, URDF)
Before this commit: robot baxter, 49 links, 48 joints
Links:
- link left_gripper: geometry collision cylinder length=0.1 radius=0.0275; visual box size=0.01 0.01 0.01
- link right_gripper: geometry collision cylinder length=0.1 radius=0.0275; visual box size=0.01 0.01 0.01

Commit message: Brought in Josh URDF

File: baxter_description/urdf/baxter.urdf (robot description, URDF)
Before this commit: robot baxter, 49 links, 48 joints
Links:
- added link block, mass 0.0001; collision box size=0.05 0.05 0.05; visual box size=0.05 0.05 0.05
- added link left_gripper_left, mass 0.0001; collision box size=0.02 0.01 0.1; visual box size=0.02 0.01 0.1
- added link left_gripper_right, mass 0.0001; collision box size=0.02 0.01 0.1; visual box size=0.02 0.01 0.1
- added link right_gripper_left, mass 0.0001; collision box size=0.02 0.01 0.1; visual box size=0.02 0.01 0.1
- added link right_gripper_right, mass 0.0001; collision box size=0.02 0.01 0.1; visual box size=0.02 0.01 0.1
- link left_gripper: geometry visual box size=0.01 0.01 0.01
- link right_gripper: geometry visual box size=0.01 0.01 0.01
Joints:
- added joint block: type fixed, parent left_gripper, child block, origin xyz=0.0 0.0 0.05 rpy=0 0 0
- added joint left_endpoint_left: type fixed, parent left_gripper, child left_gripper_left, origin xyz=0.0 0.05 0.05 rpy=0 0 0
- added joint left_endpoint_right: type fixed, parent left_gripper, child left_gripper_right, origin xyz=0.0 -0.05 0.05 rpy=0 0 0
- added joint right_endpoint_left: type fixed, parent right_gripper, child right_gripper_left, origin xyz=0.0 0.05 0.05 rpy=0 0 0
- added joint right_endpoint_right: type fixed, parent right_gripper, child right_gripper_right, origin xyz=0.0 -0.05 0.05 rpy=0 0 0

Commit message: Revert "Brought in Josh URDF"
This reverts commit ea7684a66401c413b5c3cda0f40d8a149b42786d.

File: baxter_description/urdf/baxter.urdf (robot description, URDF)
Before this commit: robot baxter, 54 links, 53 joints
Links:
- removed link block
- removed link left_gripper_left
- removed link left_gripper_right
- removed link right_gripper_left
- removed link right_gripper_right
- link left_gripper: geometry collision cylinder length=0.1 radius=0.0275; visual box size=0.01 0.01 0.01
- link right_gripper: geometry collision cylinder length=0.1 radius=0.0275; visual box size=0.01 0.01 0.01
Joints:
- removed joint block
- removed joint left_endpoint_left
- removed joint left_endpoint_right
- removed joint right_endpoint_left
- removed joint right_endpoint_right
